File: hardware/turbocan.kicad_sch (KiCad schematic)
At the start: 88 parts

Commit message: add solder jumper to probe supply (to select between 5v and 24v for PINDA)
Parts:
- added JP1: (no value), symbol Jumper:Jumper_3_Bridged12
Connections:
- net +24V: now also JP1.3 (B); no longer J14.1 (Pin_1)
- net +5V: now also JP1.1 (A)
- new net: J14.1 (Pin_1), JP1.2 (C)
Changed lines of the file:
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@@
     (stroke (width 0) (type default) (color 0 0 0 0))
   )
+  (wire (pts (xy 118.11 60.96) (xy 118.11 57.15))
+    (stroke (width 0) (type default) (color 0 0 0 0))
+  )
   (wire (pts (xy 176.53 115.57) (xy 173.99 115.57))
     (stroke (width 0) (type default) (color 0 0 0 0))
@@
     (stroke (width 0) (type default) (color 0 0 0 0))
   )
+  (wire (pts (xy 118.11 57.15) (xy 125.73 57.15))
+    (stroke (width 0) (type default) (color 0 0 0 0))
+  )
   (wire (pts (xy 24.13 33.02) (xy 24.13 38.1))
     (stroke (width 0) (type default) (color 0 0 0 0))
@@
     (stroke (width 0) (type default) (color 0 0 0 0))
   )
-  (wire (pts (xy 125.73 57.15) (xy 115.57 57.15))
-    (stroke (width 0) (type default) (color 0 0 0 0))
-  )
   (wire (pts (xy 190.5 39.37) (xy 193.04 39.37))
     (stroke (width 0) (type default) (color 0 0 0 0))
@@
     (stroke (width 0) (type default) (color 0 0 0 0))
   )
+  (wire (pts (xy 101.6 57.15) (xy 102.87 57.15))
+    (stroke (width 0) (type default) (color 0 0 0 0))
+  )
   (wire (pts (xy 250.19 119.38) (xy 252.73 119.38))
     (stroke (width 0) (type default) (color 0 0 0 0))
@@
     (stroke (width 0) (type default) (color 0 0 0 0))
   )
+  (wire (pts (xy 109.22 60.96) (xy 118.11 60.96))
+    (stroke (width 0) (type default) (color 0 0 0 0))
+  )
   (wire (pts (xy 143.51 171.45) (xy 148.59 171.45))
     (stroke (width 0) (type default) (color 0 0 0 0))
@@
     (pin "1")
   )
+  (symbol (lib_id "Jumper:Jumper_3_Bridged12") (at 109.22 57.15 0) (unit 1)
+    (in_bom yes) (on_board yes) (fields_autoplaced)
+    (property "Reference" "JP1" (id 0) (at 109.22 50.8 0))
+    (property "Value" "" (id 1) (at 109.22 53.34 0))
+    (property "Footprint" "" (id 2) (at 109.22 57.15 0)
+      (effects (font (size 1.27 1.27)) hide)
+    )
+    (property "Datasheet" "~" (id 3) (at 109.22 57.15 0)
+      (effects (font (size 1.27 1.27)) hide)
+    )
+    (pin "1")
+    (pin "2")
+    (pin "3")
+  )
+  (symbol (lib_id "archive:power_+5V") (at 101.6 57.15 0) (unit 1)
+    (in_bom yes) (on_board yes)
+    (property "Reference" "#PWR016" (id 0) (at 101.6 60.96 0)
+      (effects (font (size 1.27 1.27)) hide)
+    )
+    (property "Value" "+5V" (id 1) (at 101.981 52.7558 0))
+    (property "Footprint" "" (id 2) (at 101.6 57.15 0)
+      (effects (font (size 1.27 1.27)) hide)
+    )
+    (property "Datasheet" "" (id 3) (at 101.6 57.15 0)
+      (effects (font (size 1.27 1.27)) hide)
+    )
+    (pin "1")
+  )
   (sheet_instances
     (path "/" (page "1"))
@@
       (reference "#PWR015") (unit 1) (value "+3.3V") (footprint "")
     )
+    (path "/fa1d0408-ba61-4506-8f85-f35aebcae5a7"
+      (reference "#PWR016") (unit 1) (value "+5V") (footprint "")
+    )
     (path "/00000000-0000-0000-0000-000060c1e7ad"
       (reference "#PWR017") (unit 1) (value "+3.3V") (footprint "")
@@
       (reference "J14") (unit 1) (value "PROBE") (footprint "Connector_JST:JST_XH_B3B-XH-A_1x03_P2.50mm_Vertical")
     )
+    (path "/bec6e4e8-f492-4d4d-99a3-c79b3906d702"
+      (reference "JP1") (unit 1) (value "VPROBE") (footprint "Jumper:SolderJumper-3_P1.3mm_Bridged12_RoundedPad1.0x1.5mm")
+    )
     (path "/00000000-0000-0000-0000-00006071d843"
